Commit message: move caster component to xacro that component/caster.xacro

File: urdf/d03x.urdf (robot description, URDF)
Before this commit: robot d03x, 8 links, 7 joints
Links:
- removed link caster_housing_left_link
- removed link caster_housing_right_link
- removed link caster_wheel_left_link
- removed link caster_wheel_right_link
- added link left_caster_housing_link; collision mesh filename=package://d03_description/meshes/caster_housing.stl scale=0.001 0.001 0.001; visual mesh filename=package://d03_description/meshes/caster_housing.stl scale=0.001 0.001 0.001
- added link left_caster_wheel_link; collision mesh filename=package://d03_description/meshes/caster_wheel.stl scale=0.001 0.001 0.001; visual mesh filename=package://d03_description/meshes/caster_wheel.stl scale=0.001 0.001 0.001
- added link right_caster_housing_link; collision mesh filename=package://d03_description/meshes/caster_housing.stl scale=0.001 0.001 0.001; visual mesh filename=package://d03_description/meshes/caster_housing.stl scale=0.001 0.001 0.001
- added link right_caster_wheel_link; collision mesh filename=package://d03_description/meshes/caster_wheel.stl scale=0.001 0.001 0.001; visual mesh filename=package://d03_description/meshes/caster_wheel.stl scale=0.001 0.001 0.001
Joints:
- removed joint caster_housing_left_joint
- removed joint caster_housing_right_joint
- removed joint caster_wheel_left_joint
- removed joint caster_wheel_right_joint
- added joint left_caster_housing_joint: type continuous, parent base_link, child left_caster_housing_link, origin xyz=-0.14 0.14 0.089837 rpy=0 0 3.1415926, axis 0 0 1
- added joint left_caster_wheel_joint: type continuous, parent left_caster_housing_link, child left_caster_wheel_link, origin xyz=0.031 0.0 -0.052 rpy=0 0 0, axis 0 1 0
- added joint right_caster_housing_joint: type continuous, parent base_link, child right_caster_housing_link, origin xyz=-0.14 -0.14 0.089837 rpy=0 0 3.1415926, axis 0 0 1
- added joint right_caster_wheel_joint: type continuous, parent right_caster_housing_link, child right_caster_wheel_link, origin xyz=0.031 0.0 -0.052 rpy=0 0 0, axis 0 1 0
